Commit message: Update simple_box_robot.urdf

File: CAD/EdyMobile_URDF_screencast_ROS/URDF_screencast_ROS/urdf/simple_box_robot.urdf (robot description, URDF)
Before this commit: robot simple_box_robot, 1 links, 0 joints
Links:
- link base_link: geometry collision box size=0.3 0.174 0.13; visual box size=0.3 0.174 0.13
